Commit message: updated regenerated urdf

File: urdf/shadow_drone.urdf (robot description, URDF)
Before this commit: robot shadow_drone, 3 links, 2 joints
Links:
- added link battery_link; visual box size=0.07 0.035 0.025
- added link motor_front_left; visual cylinder length=0.03 radius=0.014
- added link motor_front_right; visual cylinder length=0.03 radius=0.014
- added link motor_rear_left; visual cylinder length=0.03 radius=0.014
- added link motor_rear_right; visual cylinder length=0.03 radius=0.014
- added link stack_link; visual box size=0.09 0.065 0.04
- link base_link: mass 1.0 -> 0.15; geometry collision box size=0.25 0.25 0.02; visual box size=0.25 0.25 0.02
- link camera_link: geometry visual box size=0.025 0.025 0.015
- link lidar_link: geometry visual cylinder length=0.04 radius=0.035
Joints:
- added joint battery_joint: type fixed, parent base_link, child battery_link, origin xyz=0 0 -0.04 rpy=0 0 0
- added joint motor_front_left_joint: type fixed, parent base_link, child motor_front_left, origin xyz=-0.125 0.125 0.0 rpy=0 0 0
- added joint motor_front_right_joint: type fixed, parent base_link, child motor_front_right, origin xyz=0.125 0.125 0.0 rpy=0 0 0
- added joint motor_rear_left_joint: type fixed, parent base_link, child motor_rear_left, origin xyz=-0.125 -0.125 0.0 rpy=0 0 0
- added joint motor_rear_right_joint: type fixed, parent base_link, child motor_rear_right, origin xyz=0.125 -0.125 0.0 rpy=0 0 0
- added joint stack_joint: type fixed, parent base_link, child stack_link, origin xyz=0 0 0.04 rpy=0 0 0
- joint camera_joint: origin xyz=0.1 0 0 rpy=0 0 0 -> xyz=0.06 0 0.0 rpy=0 0 0; parent base_link -> stack_link
- joint lidar_joint: origin xyz=0 0 0.1 rpy=0 0 0 -> xyz=0 0 0.05 rpy=0 0 0; parent base_link -> stack_link
